File: board/ethernet.kicad_sch (KiCad schematic)
At the start: 16 parts, among them Con1 74990111215A_RJ45

Commit message: pcb layout
Parts:
- Con1: footprint (none) -> v3s:74990111215A_RJ45
- L4: value 10u -> FB; footprint (none) -> Resistor_SMD:R_0805_2012Metric
- R30, R31, R32, R33: value 10 -> 49.9
Connections:
- net GND: now also Con1.13 (CASE)
Changed lines of the file:
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@@
   (junction (at 84.455 78.74) (diameter 0) (color 0 0 0 0)
   )
+  (junction (at 83.82 99.06) (diameter 0) (color 0 0 0 0)
+  )
   (junction (at 60.96 67.945) (diameter 0) (color 0 0 0 0)
   )
@@
     (stroke (width 0) (type default) (color 0 0 0 0))
   )
+  (wire (pts (xy 83.82 99.06) (xy 83.82 108.712))
+    (stroke (width 0) (type default) (color 0 0 0 0))
+  )
   (wire (pts (xy 121.92 81.28) (xy 121.92 102.235))
     (stroke (width 0) (type default) (color 0 0 0 0))
@@
     (stroke (width 0) (type default) (color 0 0 0 0))
   )
-  (wire (pts (xy 121.92 81.28) (xy 124.46 81.28))
+  (wire (pts (xy 121.92 81.28) (xy 157.48 81.28))
     (stroke (width 0) (type default) (color 0 0 0 0))
   )
@@
     (stroke (width 0) (type default) (color 0 0 0 0))
   )
-  (wire (pts (xy 139.7 88.9) (xy 142.24 88.9))
+  (wire (pts (xy 139.7 88.9) (xy 157.48 88.9))
     (stroke (width 0) (type default) (color 0 0 0 0))
   )
@@
     (stroke (width 0) (type default) (color 0 0 0 0))
   )
+  (wire (pts (xy 83.82 99.06) (xy 90.17 99.06))
+    (stroke (width 0) (type default) (color 0 0 0 0))
+  )
   (wire (pts (xy 84.455 78.74) (xy 84.455 76.2))
     (stroke (width 0) (type default) (color 0 0 0 0))
@@
     (stroke (width 0) (type default) (color 0 0 0 0))
   )
-  (wire (pts (xy 130.81 86.36) (xy 133.35 86.36))
+  (wire (pts (xy 130.81 86.36) (xy 157.48 86.36))
     (stroke (width 0) (type default) (color 0 0 0 0))
   )
@@
     (stroke (width 0) (type default) (color 0 0 0 0))
   )
-  (wire (pts (xy 113.03 78.74) (xy 115.57 78.74))
+  (wire (pts (xy 113.03 78.74) (xy 157.48 78.74))
     (stroke (width 0) (type default) (color 0 0 0 0))
   )
@@
     (stroke (width 0) (type default) (color 0 0 0 0))
   )
-  (wire (pts (xy 83.82 100.33) (xy 83.82 96.52))
+  (wire (pts (xy 83.82 96.52) (xy 83.82 99.06))
     (stroke (width 0) (type default) (color 0 0 0 0))
   )
@@
     (stroke (width 0) (type default) (color 0 0 0 0))
   )
-  (hierarchical_label "RD+" (shape input) (at 133.35 86.36 0)
+  (hierarchical_label "RD+" (shape input) (at 157.48 86.36 0)
     (effects (font (size 1.27 1.27)) (justify left))
   )
@@
     (effects (font (size 1.27 1.27)) (justify left))
   )
-  (hierarchical_label "TD-" (shape input) (at 124.46 81.28 0)
+  (hierarchical_label "TD-" (shape input) (at 157.48 81.28 0)
     (effects (font (size 1.27 1.27)) (justify left))
   )
-  (hierarchical_label "RD-" (shape input) (at 142.24 88.9 0)
+  (hierarchical_label "RD-" (shape input) (at 157.48 88.9 0)
     (effects (font (size 1.27 1.27)) (justify left))
   )
-  (hierarchical_label "TD+" (shape input) (at 115.57 78.74 0)
+  (hierarchical_label "TD+" (shape input) (at 157.48 78.74 0)
     (effects (font (size 1.27 1.27)) (justify left))
   )
   (symbol (lib_id "Device:R_Small") (at 145.415 96.52 90) (unit 1)
     (in_bom yes) (on_board yes)
-    (property "Reference" "R34" (id 0) (at 144.145 99.06 90))
-    (property "Value" "1k" (id 1) (at 146.685 99.06 90))
+    (property "Reference" "R34" (id 0) (at 143.51 98.806 90))
+    (property "Value" "1k" (id 1) (at 147.066 98.806 90))
     (property "Footprint" "Resistor_SMD:R_0603_1608Metric" (id 2) (at 145.415 96.52 0)
       (effects (font (size 1.27 1.27)) hide)
@@
   (symbol (lib_id "Device:R_Small") (at 149.225 93.98 90) (unit 1)
     (in_bom yes) (on_board yes)
-    (property "Reference" "R35" (id 0) (at 147.955 91.44 90))
-    (property "Value" "1k" (id 1) (at 150.495 91.44 90))
+    (property "Reference" "R35" (id 0) (at 147.32 91.694 90))
+    (property "Value" "1k" (id 1) (at 150.876 91.694 90))
     (property "Footprint" "Resistor_SMD:R_0603_1608Metric" (id 2) (at 149.225 93.98 0)
       (effects (font (size 1.27 1.27)) hide)
@@
       (effects (font (size 1.27 1.27)) (justify right))
     )
-    (property "Value" "10u" (id 1) (at 61.595 64.7699 0)
+    (property "Value" "FB" (id 1) (at 61.595 64.7699 0)
       (effects (font (size 1.27 1.27)) (justify right))
     )
-    (property "Footprint" "" (id 2) (at 60.96 63.5 0)
+    (property "Footprint" "Resistor_SMD:R_0805_2012Metric" (id 2) (at 60.96 63.5 0)
       (effects (font (size 1.27 1.27)) hide)
     )
@@
       (effects (font (size 1.27 1.27)) (justify left))
     )
-    (property "Value" "10" (id 1) (at 140.97 73.66 0)
+    (property "Value" "49.9" (id 1) (at 140.97 73.66 0)
       (effects (font (size 1.27 1.27)) (justify left))
     )
@@
     (in_bom yes) (on_board yes)
     (property "Reference" "Con1" (id 0) (at 99.06 74.93 0))
-    (property "Value" "74990111215A_RJ45" (id 1) (at 99.06 101.6 0))
-    (property "Footprint" "" (id 2) (at 105.41 78.74 0)
+    (property "Value" "74990111215A_RJ45" (id 1) (at 99.06 102.87 0))
+    (property "Footprint" "v3s:74990111215A_RJ45" (id 2) (at 105.41 78.74 0)
       (effects (font (size 1.27 1.27)) hide)
     )
@@
     (pin "11")
     (pin "12")
+    (pin "13")
     (pin "2")
     (pin "3")
@@
     (pin "1")
   )
-  (symbol (lib_id "power:GND") (at 83.82 100.33 0) (unit 1)
-    (in_bom yes) (on_board yes)
-    (property "Reference" "#PWR0171" (id 0) (at 83.82 106.68 0)
-      (effects (font (size 1.27 1.27)) hide)
-    )
-    (property "Value" "GND" (id 1) (at 83.82 104.14 0))
-    (property "Footprint" "" (id 2) (at 83.82 100.33 0)
-      (effects (font (size 1.27 1.27)) hide)
-    )
-    (property "Datasheet" "" (id 3) (at 83.82 100.33 0)
+  (symbol (lib_id "power:GND") (at 83.82 108.712 0) (unit 1)
+    (in_bom yes) (on_board yes)
+    (property "Reference" "#PWR0171" (id 0) (at 83.82 115.062 0)
+      (effects (font (size 1.27 1.27)) hide)
+    )
+    (property "Value" "GND" (id 1) (at 83.82 112.522 0))
+    (property "Footprint" "" (id 2) (at 83.82 108.712 0)
+      (effects (font (size 1.27 1.27)) hide)
+    )
+    (property "Datasheet" "" (id 3) (at 83.82 108.712 0)
       (effects (font (size 1.27 1.27)) hide)
     )
@@
       (effects (font (size 1.27 1.27)) (justify left))
     )
-    (property "Value" "10" (id 1) (at 132.08 73.66 0)
+    (property "Value" "49.9" (id 1) (at 132.08 73.66 0)
       (effects (font (size 1.27 1.27)) (justify left))
     )
@@
       (effects (font (size 1.27 1.27)) (justify left))
     )
-    (property "Value" "10" (id 1) (at 123.19 73.66 0)
+    (property "Value" "49.9" (id 1) (at 123.19 73.66 0)
       (effects (font (size 1.27 1.27)) (justify left))
     )
@@
       (effects (font (size 1.27 1.27)) (justify left))
     )
-    (property "Value" "10" (id 1) (at 114.3 73.66 0)
-      (effects (font (size 1.27 1.27)) (justify left))
-    )
+    (property "Value" "49.9" (id 1) (at 114.3 73.66 0)
+      (effects (font (size 1.27 1.27)) (justify left))
+    )
