File: board/sdCard.kicad_sch (KiCad schematic)
At the start: 8 parts, among them U6 693072010801

Commit message: pcb layout
Parts:
- R15, R16, R17, R18, R19: value 4.7k -> 47k
- U6: footprint (none) -> v3s:693072010801
Changed lines of the file:
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@@
     (property "Reference" "U6" (id 0) (at 47.625 44.45 0))
     (property "Value" "693072010801" (id 1) (at 47.625 46.99 0))
-    (property "Footprint" "" (id 2) (at 50.8 57.15 0)
+    (property "Footprint" "v3s:693072010801" (id 2) (at 50.8 57.15 0)
       (effects (font (size 1.27 1.27)) hide)
     )
@@
       (effects (font (size 1.27 1.27)) (justify left))
     )
-    (property "Value" "4.7k" (id 1) (at 118.11 36.83 0)
+    (property "Value" "47k" (id 1) (at 118.11 36.83 0)
       (effects (font (size 1.27 1.27)) (justify left))
     )
@@
       (effects (font (size 1.27 1.27)) (justify left))
     )
-    (property "Value" "4.7k" (id 1) (at 87.63 36.83 0)
+    (property "Value" "47k" (id 1) (at 87.63 36.83 0)
       (effects (font (size 1.27 1.27)) (justify left))
     )
@@
       (effects (font (size 1.27 1.27)) (justify left))
     )
-    (property "Value" "4.7k" (id 1) (at 102.87 36.83 0)
+    (property "Value" "47k" (id 1) (at 102.87 36.83 0)
       (effects (font (size 1.27 1.27)) (justify left))
     )
@@
       (effects (font (size 1.27 1.27)) (justify left))
     )
-    (property "Value" "4.7k" (id 1) (at 95.25 36.83 0)
+    (property "Value" "47k" (id 1) (at 95.25 36.83 0)
       (effects (font (size 1.27 1.27)) (justify left))
     )
@@
       (effects (font (size 1.27 1.27)) (justify left))
     )
-    (property "Value" "4.7k" (id 1) (at 110.49 36.83 0)
+    (property "Value" "47k" (id 1) (at 110.49 36.83 0)
       (effects (font (size 1.27 1.27)) (justify left))
     )
