File: board/CPU.kicad_sch (KiCad schematic)
At the start: 32 parts

Commit message: schematic update, choose components, creeate footprints
Parts:
- C1, C2: renamed from C?; value 18p -> 9p; footprint (none) -> Capacitor_SMD:C_0603_1608Metric
- C10, C11, C12, C13, C3, C4, C5, C8, C9: renamed from C?; footprint (none) -> Capacitor_SMD:C_0603_1608Metric
- C6, C7: renamed from C?; value 18p -> 6p; footprint (none) -> Capacitor_SMD:C_0603_1608Metric
- R1: renamed from R?; footprint Resistor_SMD:R_0805_2012Metric -> Resistor_SMD:R_0603_1608Metric
- R2, R3, R4, R5, R6, R7, R8: renamed from R?; footprint (none) -> Resistor_SMD:R_0603_1608Metric
- U1: renamed from U?; footprint (none) -> Package_QFP:LQFP-128_14x14mm_P0.4mm
- Y1: renamed from Y?; value 32KHz -> SC32S-7PF20PPM; footprint (none) -> v3s:SC32S-7PF20PPM
- Y2: renamed from Y?; value 24MHz -> XRCGB24M000F2P00R0; footprint (none) -> v3s:XRCGB24M000F2P00R0
Connections:
- net CPU_PG4: now reaches U1.1 (PG4)
- net CPU_PE20: now reaches U1.10 (PE20)
- net CPU_PF6: now reaches U1.100 (PF6)
- net CPU_PE19: now reaches U1.11 (PE19)
- net CPU_PG5: now reaches U1.128 (PG5)
- net CPU_PE18: now reaches U1.13 (PE18)
- net CPU_PE17: now reaches U1.14 (PE17)
- net CPU_PE16: now reaches U1.15 (PE16)
- net CPU_PE15: now reaches U1.16 (PE15)
- net CPU_PE14: now reaches U1.17 (PE14)
- net CPU_PE13: now reaches U1.18 (PE13)
- net CPU_PG3: now reaches U1.2 (PG3)
- net CPU_PE12: now reaches U1.22 (PE12)
- net CPU_PE11: now reaches U1.23 (PE11)
- net CPU_PE10: now reaches U1.24 (PE10)
- net CPU_PE9: now reaches U1.27 (PE9)
- net CPU_PE8: now reaches U1.28 (PE8)
- net CPU_PG2: now reaches U1.3 (PG2)
- net CPU_PE7: now reaches U1.30 (PE7)
- net CPU_PE6: now reaches U1.31 (PE6)
- net CPU_PE5: now reaches U1.32 (PE5)
- net CPU_PE4: now reaches U1.33 (PE4)
- net CPU_PE3: now reaches U1.34 (PE3)
- net CPU_PE2: now reaches U1.35 (PE2)
- net CPU_PE1: now reaches U1.36 (PE1)
- net CPU_PE0: now reaches U1.37 (PE0)
- net CPU_PB0: now reaches U1.39 (PB0)
- net CPU_PG1: now reaches U1.4 (PG1)
- net CPU_PB1: now reaches U1.40 (PB1)
- net CPU_PB2: now reaches U1.41 (PB2)
- net CPU_PB3: now reaches U1.42 (PB3)
- net CPU_PB4: now reaches U1.43 (PB4)
- net CPU_PB5: now reaches U1.44 (PB5)
- net CPU_PB6: now reaches U1.45 (PB6)
- net CPU_PB7: now reaches U1.46 (PB7)
- net UART0_TX: now reaches U1.48 (PB8)
- net UART0_RX: now reaches U1.49 (PB9)
- net CPU_PG0: now reaches U1.5 (PG0)
- net CPU_PC0: now reaches U1.52 (PC0)
- net CPU_PC1: now reaches U1.53 (PC1)
- net CPU_PC2: now reaches U1.54 (PC2)
- net CPU_PC3: now reaches U1.55 (PC3)
- net CPU_PE24: now reaches U1.6 (PE24)
- net CPU_PE23: now reaches U1.7 (PE23)
- net CPU_PE22: now reaches U1.8 (PE22)
- net CPU_PE21: now reaches U1.9 (PE21)

Commit message: pcb layout
Parts:
- removed C9: 10u, Capacitor_SMD:C_0603_1608Metric, symbol Device:C_Small
- C11: value 10u -> 1u
- U1: footprint Package_QFP:LQFP-128_14x14mm_P0.4mm -> v3s:LQFP-128_14x14mm_P0.4mm_EP8x8mm
Connections:
- net USB_DN: now reaches U1.110 (USB_DM)
- net USB_DP: now reaches U1.111 (USB_DP)
- no-connect marks 15 -> 13
Changed lines of the file:
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@@
   (junction (at 121.92 120.65) (diameter 0) (color 0 0 0 0)
   )
-  (no_connect (at 177.8 121.92))
-  (no_connect (at 177.8 124.46))
   (no_connect (at 177.8 69.85))
   (no_connect (at 177.8 67.31))
@@
     (stroke (width 0) (type default) (color 0 0 0 0))
   )
+  (wire (pts (xy 177.8 121.92) (xy 181.61 121.92))
+    (stroke (width 0) (type default) (color 0 0 0 0))
+  )
   (wire (pts (xy 111.76 97.79) (xy 121.92 97.79))
     (stroke (width 0) (type default) (color 0 0 0 0))
@@
     (stroke (width 0) (type default) (color 0 0 0 0))
   )
+  (wire (pts (xy 177.8 124.46) (xy 181.61 124.46))
+    (stroke (width 0) (type default) (color 0 0 0 0))
+  )
   (wire (pts (xy 44.45 191.77) (xy 49.53 191.77))
     (stroke (width 0) (type default) (color 0 0 0 0))
@@
     (effects (font (size 1.27 1.27)) (justify left))
   )
+  (hierarchical_label "USB_DN" (shape input) (at 181.61 121.92 0)
+    (effects (font (size 1.27 1.27)) (justify left))
+  )
   (hierarchical_label "CPU_PE20" (shape input) (at 39.37 109.22 0)
     (effects (font (size 1.27 1.27)) (justify left))
@@
   )
   (hierarchical_label "CPU_PE21" (shape input) (at 39.37 111.76 0)
+    (effects (font (size 1.27 1.27)) (justify left))
+  )
+  (hierarchical_label "USB_DP" (shape input) (at 181.61 124.46 0)
     (effects (font (size 1.27 1.27)) (justify left))
   )
@@
     (pin "1")
   )
-  (symbol (lib_name "V3S_3") (lib_id "v3s:V3S") (at 74.93 167.64 0) (mirror y) (unit 3)
+  (symbol (lib_id "v3s:V3S") (at 74.93 167.64 0) (mirror y) (unit 3)
     (in_bom yes) (on_board yes) (fields_autoplaced)
     (property "Reference" "U1" (id 0) (at 67.31 160.02 0))
     (property "Value" "V3S" (id 1) (at 67.31 162.56 0))
-    (property "Footprint" "Package_QFP:LQFP-128_14x14mm_P0.4mm" (id 2) (at 74.93 218.44 0)
+    (property "Footprint" "v3s:LQFP-128_14x14mm_P0.4mm_EP8x8mm" (id 2) (at 74.93 218.44 0)
       (effects (font (size 1.27 1.27)) hide)
     )
@@
     (pin "2")
   )
-  (symbol (lib_id "Device:C_Small") (at 184.15 68.58 0) (unit 1)
-    (in_bom yes) (on_board yes) (fields_autoplaced)
-    (property "Reference" "C9" (id 0) (at 186.69 67.3162 0)
-      (effects (font (size 1.27 1.27)) (justify left))
-    )
-    (property "Value" "10u" (id 1) (at 186.69 69.8562 0)
-      (effects (font (size 1.27 1.27)) (justify left))
-    )
-    (property "Footprint" "Capacitor_SMD:C_0603_1608Metric" (id 2) (at 184.15 68.58 0)
-      (effects (font (size 1.27 1.27)) hide)
-    )
-    (property "Datasheet" "~" (id 3) (at 184.15 68.58 0)
-      (effects (font (size 1.27 1.27)) hide)
-    )
-    (pin "1")
-    (pin "2")
-  )
   (symbol (lib_id "Device:R_Small") (at 213.36 68.58 0) (unit 1)
     (in_bom yes) (on_board yes) (fields_autoplaced)
@@
     (pin "1")
   )
-  (symbol (lib_name "V3S_5") (lib_id "v3s:V3S") (at 175.26 17.78 0) (mirror y) (unit 8)
+  (symbol (lib_id "v3s:V3S") (at 175.26 17.78 0) (mirror y) (unit 8)
     (in_bom yes) (on_board yes)
     (property "Reference" "U1" (id 0) (at 161.29 13.97 0))
     (property "Value" "V3S" (id 1) (at 172.72 13.97 0))
-    (property "Footprint" "Package_QFP:LQFP-128_14x14mm_P0.4mm" (id 2) (at 175.26 68.58 0)
+    (property "Footprint" "v3s:LQFP-128_14x14mm_P0.4mm_EP8x8mm" (id 2) (at 175.26 68.58 0)
       (effects (font (size 1.27 1.27)) hide)
     )
@@
     (pin "80")
   )
-  (symbol (lib_name "V3S_8") (lib_id "v3s:V3S") (at 31.75 17.78 0) (mirror y) (unit 2)
+  (symbol (lib_id "v3s:V3S") (at 31.75 17.78 0) (mirror y) (unit 2)
     (in_bom yes) (on_board yes)
     (property "Reference" "U1" (id 0) (at 16.51 13.97 0))
     (property "Value" "V3S" (id 1) (at 30.48 13.97 0))
-    (property "Footprint" "Package_QFP:LQFP-128_14x14mm_P0.4mm" (id 2) (at 31.75 68.58 0)
+    (property "Footprint" "v3s:LQFP-128_14x14mm_P0.4mm_EP8x8mm" (id 2) (at 31.75 68.58 0)
       (effects (font (size 1.27 1.27)) hide)
     )
@@
     (pin "1")
   )
-  (symbol (lib_name "V3S_1") (lib_id "v3s:V3S") (at 175.26 54.61 0) (mirror y) (unit 6)
+  (symbol (lib_id "v3s:V3S") (at 175.26 54.61 0) (mirror y) (unit 6)
     (in_bom yes) (on_board yes)
     (property "Reference" "U1" (id 0) (at 162.56 50.8 0))
     (property "Value" "V3S" (id 1) (at 172.72 50.8 0))
-    (property "Footprint" "Package_QFP:LQFP-128_14x14mm_P0.4mm" (id 2) (at 175.26 105.41 0)
+    (property "Footprint" "v3s:LQFP-128_14x14mm_P0.4mm_EP8x8mm" (id 2) (at 175.26 105.41 0)
       (effects (font (size 1.27 1.27)) hide)
     )
@@
     (property "Reference" "U1" (id 0) (at 115.57 172.72 0))
     (property "Value" "V3S" (id 1) (at 127 172.72 0))
-    (property "Footprint" "Package_QFP:LQFP-128_14x14mm_P0.4mm" (id 2) (at 129.54 227.33 0)
+    (property "Footprint" "v3s:LQFP-128_14x14mm_P0.4mm_EP8x8mm" (id 2) (at 129.54 227.33 0)
       (effects (font (size 1.27 1.27)) hide)
     )
@@
       (effects (font (size 1.27 1.27)) (justify left))
     )
-    (property "Value" "10u" (id 1) (at 207.01 69.8562 0)
+    (property "Value" "1u" (id 1) (at 207.01 69.8562 0)
       (effects (font (size 1.27 1.27)) (justify left))
     )
@@
     (pin "2")
   )
-  (symbol (lib_name "V3S_2") (lib_id "v3s:V3S") (at 31.75 171.45 0) (mirror y) (unit 7)
+  (symbol (lib_id "v3s:V3S") (at 31.75 171.45 0) (mirror y) (unit 7)
     (in_bom yes) (on_board yes)
     (property "Reference" "U1" (id 0) (at 19.05 167.64 0))
     (property "Value" "V3S" (id 1) (at 29.21 167.64 0))
-    (property "Footprint" "Package_QFP:LQFP-128_14x14mm_P0.4mm" (id 2) (at 31.75 222.25 0)
+    (property "Footprint" "v3s:LQFP-128_14x14mm_P0.4mm_EP8x8mm" (id 2) (at 31.75 222.25 0)
       (effects (font (size 1.27 1.27)) hide)
     )
@@
     (pin "80")
   )
-  (symbol (lib_name "V3S_6") (lib_id "v3s:V3S") (at 175.26 119.38 0) (mirror y) (unit 5)
+  (symbol (lib_id "v3s:V3S") (at 175.26 119.38 0) (mirror y) (unit 5)
     (in_bom yes) (on_board yes)
     (property "Reference" "U1" (id 0) (at 167.64 111.76 0))
     (property "Value" "V3S" (id 1) (at 167.64 114.3 0))
-    (property "Footprint" "Package_QFP:LQFP-128_14x14mm_P0.4mm" (id 2) (at 175.26 170.18 0)
+    (property "Footprint" "v3s:LQFP-128_14x14mm_P0.4mm_EP8x8mm" (id 2) (at 175.26 170.18 0)
       (effects (font (size 1.27 1.27)) hide)
     )
@@
     (pin "1")
   )
-  (symbol (lib_name "V3S_7") (lib_id "v3s:V3S") (at 109.22 80.01 0) (mirror y) (unit 9)
+  (symbol (lib_id "v3s:V3S") (at 109.22 80.01 0) (mirror y) (unit 9)
     (in_bom yes) (on_board yes) (fields_autoplaced)
     (property "Reference" "U1" (id 0) (at 101.6 72.39 0))
     (property "Value" "V3S" (id 1) (at 101.6 74.93 0))
-    (property "Footprint" "Package_QFP:LQFP-128_14x14mm_P0.4mm" (id 2) (at 109.22 130.81 0)
+    (property "Footprint" "v3s:LQFP-128_14x14mm_P0.4mm_EP8x8mm" (id 2) (at 109.22 130.81 0)
       (effects (font (size 1.27 1.27)) hide)
     )
@@
   (symbol (lib_id "power:+1V8") (at 120.65 44.45 0) (unit 1)
     (in_bom yes) (on_board yes)
-    (property "Reference" "#PWR?" (id 0) (at 120.65 48.26 0)
+    (property "Reference" "#PWR0177" (id 0) (at 120.65 48.26 0)
       (effects (font (size 1.27 1.27)) hide)
     )
@@
     (pin "2")
   )
-  (symbol (lib_name "V3S_4") (lib_id "v3s:V3S") (at 109.22 17.78 0) (mirror y) (unit 1)
+  (symbol (lib_id "v3s:V3S") (at 109.22 17.78 0) (mirror y) (unit 1)
     (in_bom yes) (on_board yes)
     (property "Reference" "U1" (id 0) (at 90.17 13.97 0))
     (property "Value" "V3S" (id 1) (at 106.68 13.97 0))
-    (property "Footprint" "Package_QFP:LQFP-128_14x14mm_P0.4mm" (id 2) (at 109.22 68.58 0)
-      (effects (font (size 1.27 1.27)) hide)
-    )
+    (property "Footprint" "v3s:LQFP-128_14x14mm_P0.4mm_EP8x8mm" (id 2) (at 109.22 68.58 0)
+      (effects (font (size 1.27 1.27)) hide)
+    )

Commit message: update layout
Parts:
- removed C13: 100n, Capacitor_SMD:C_0603_1608Metric, symbol Device:C_Small
- removed R8: 200k 1%, Resistor_SMD:R_0603_1608Metric, symbol Device:R_Small
Connections:
- net LRADC: no longer names the net of U1.112 (LRADC0)
- no-connect marks 13 -> 14
Changed lines of the file:
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@@
   (junction (at 115.57 43.18) (diameter 0) (color 0 0 0 0)
-  )
-  (junction (at 236.22 85.09) (diameter 0) (color 0 0 0 0)
   )
   (junction (at 121.92 100.33) (diameter 0) (color 0 0 0 0)
@@
   (no_connect (at 177.8 72.39))
   (no_connect (at 177.8 77.47))
+  (no_connect (at 177.8 85.09))
   (no_connect (at 177.8 33.02))
   (no_connect (at 177.8 30.48))
@@
     (stroke (width 0) (type default) (color 0 0 0 0))
   )
-  (wire (pts (xy 177.8 85.09) (xy 236.22 85.09))
-    (stroke (width 0) (type default) (color 0 0 0 0))
-  )
   (wire (pts (xy 121.92 130.81) (xy 121.92 133.35))
     (stroke (width 0) (type default) (color 0 0 0 0))
@@
     (stroke (width 0) (type default) (color 0 0 0 0))
   )
-  (wire (pts (xy 236.22 85.09) (xy 236.22 87.63))
-    (stroke (width 0) (type default) (color 0 0 0 0))
-  )
   (wire (pts (xy 180.34 87.63) (xy 180.34 90.17))
     (stroke (width 0) (type default) (color 0 0 0 0))
@@
     (stroke (width 0) (type default) (color 0 0 0 0))
   )
-  (wire (pts (xy 236.22 82.55) (xy 236.22 85.09))
-    (stroke (width 0) (type default) (color 0 0 0 0))
-  )
   (wire (pts (xy 111.76 92.71) (xy 115.57 92.71))
     (stroke (width 0) (type default) (color 0 0 0 0))
@@
     (stroke (width 0) (type default) (color 0 0 0 0))
   )
-  (wire (pts (xy 236.22 92.71) (xy 236.22 93.98))
-    (stroke (width 0) (type default) (color 0 0 0 0))
-  )
-  (wire (pts (xy 236.22 85.09) (xy 250.19 85.09))
-    (stroke (width 0) (type default) (color 0 0 0 0))
-  )
   (wire (pts (xy 120.65 44.45) (xy 120.65 45.72))
     (stroke (width 0) (type default) (color 0 0 0 0))
@@
     (stroke (width 0) (type default) (color 0 0 0 0))
   )
-  (wire (pts (xy 236.22 74.93) (xy 236.22 77.47))
-    (stroke (width 0) (type default) (color 0 0 0 0))
-  )
   (wire (pts (xy 34.29 111.76) (xy 39.37 111.76))
     (stroke (width 0) (type default) (color 0 0 0 0))
@@
     (stroke (width 0) (type default) (color 0 0 0 0))
   )
+  (label "CPU_RESET" (at 137.795 176.53 0)
+    (effects (font (size 1.27 1.27)) (justify left bottom))
+  )
   (hierarchical_label "CPU_PC0" (shape input) (at 39.37 45.72 0)
     (effects (font (size 1.27 1.27)) (justify left))
@@
   )
   (hierarchical_label "CPU_PB2" (shape input) (at 39.37 22.86 0)
-    (effects (font (size 1.27 1.27)) (justify left))
-  )
-  (hierarchical_label "LRADC" (shape input) (at 250.19 85.09 0)
     (effects (font (size 1.27 1.27)) (justify left))
   )
@@
     (pin "2")
   )
-  (symbol (lib_id "Device:C_Small") (at 236.22 90.17 0) (unit 1)
-    (in_bom yes) (on_board yes) (fields_autoplaced)
-    (property "Reference" "C13" (id 0) (at 238.76 88.9062 0)
-      (effects (font (size 1.27 1.27)) (justify left))
-    )
-    (property "Value" "100n" (id 1) (at 238.76 91.4462 0)
-      (effects (font (size 1.27 1.27)) (justify left))
-    )
-    (property "Footprint" "Capacitor_SMD:C_0603_1608Metric" (id 2) (at 236.22 90.17 0)
-      (effects (font (size 1.27 1.27)) hide)
-    )
-    (property "Datasheet" "~" (id 3) (at 236.22 90.17 0)
-      (effects (font (size 1.27 1.27)) hide)
-    )
-    (pin "1")
-    (pin "2")
-  )
   (symbol (lib_id "power:+3V3") (at 36.83 168.91 0) (unit 1)
     (in_bom yes) (on_board yes)
@@
     (pin "2")
   )
-  (symbol (lib_id "Device:R_Small") (at 236.22 80.01 0) (unit 1)
-    (in_bom yes) (on_board yes) (fields_autoplaced)
-    (property "Reference" "R8" (id 0) (at 238.76 78.7399 0)
-      (effects (font (size 1.27 1.27)) (justify left))
-    )
-    (property "Value" "200k 1%" (id 1) (at 238.76 81.2799 0)
-      (effects (font (size 1.27 1.27)) (justify left))
-    )
-    (property "Footprint" "Resistor_SMD:R_0603_1608Metric" (id 2) (at 236.22 80.01 0)
-      (effects (font (size 1.27 1.27)) hide)
-    )
-    (property "Datasheet" "~" (id 3) (at 236.22 80.01 0)
-      (effects (font (size 1.27 1.27)) hide)
-    )
-    (pin "1")
-    (pin "2")
-  )
   (symbol (lib_id "Device:C_Small") (at 204.47 68.58 0) (unit 1)
     (in_bom yes) (on_board yes) (fields_autoplaced)
@@
     (pin "2")
   )
-  (symbol (lib_id "power:+3V3") (at 236.22 74.93 0) (unit 1)
-    (in_bom yes) (on_board yes)
-    (property "Reference" "#PWR0114" (id 0) (at 236.22 78.74 0)
-      (effects (font (size 1.27 1.27)) hide)
-    )
-    (property "Value" "+3V3" (id 1) (at 236.22 71.12 0))
-    (property "Footprint" "" (id 2) (at 236.22 74.93 0)
-      (effects (font (size 1.27 1.27)) hide)
-    )
-    (property "Datasheet" "" (id 3) (at 236.22 74.93 0)
-      (effects (font (size 1.27 1.27)) hide)
-    )
-    (pin "1")
-  )
   (symbol (lib_id "power:+3V3") (at 86.36 161.29 0) (unit 1)
     (in_bom yes) (on_board yes)
@@
       (effects (font (size 1.27 1.27)) hide)
     )
-    (pin "1")
-  )
-  (symbol (lib_id "power:GND") (at 236.22 93.98 0) (unit 1)
-    (in_bom yes) (on_board yes)
-    (property "Reference" "#PWR0116" (id 0) (at 236.22 100.33 0)
-      (effects (font (size 1.27 1.27)) hide)
-    )
-    (property "Value" "GND" (id 1) (at 236.22 97.79 0))
-    (property "Footprint" "" (id 2) (at 236.22 93.98 0)
-      (effects (font (size 1.27 1.27)) hide)
-    )
-    (property "Datasheet" "" (id 3) (at 236.22 93.98 0)
-      (effects (font (size 1.27 1.27)) hide)
-    )

Commit message: updates, finish layout, remove usb-uart
Parts:
- Y1: value SC32S-7PF20PPM -> Q13FC1350000212; footprint v3s:SC32S-7PF20PPM -> Crystal:Crystal_SMD_3215-2Pin_3.2x1.5mm
