File: board/v3s.kicad_pcb (KiCad board)
At the start: 4 copper layers, 70 x 49 mm, 123 parts, among them Con1 74990111215A_RJ45, J1 Conn_01x02, J2 629105150521, J3 Conn_02x13_Odd_Even, U1 V3S, U2 AP63200WU-7, U3 AP63200WU-7, U4 AP63200WU-7, U5 NCP114ASN300T1G, U6 693072010801, U7 CP2102N-Axx-xQFN20, Y1 SC32S-7PF20PPM, Y2 XRCGB24M000F2P00R0

Commit message: update layout
Parts:
- removed C13: 100n, Capacitor_SMD:C_0603_1608Metric
- removed J2: 629105150521, v3s:629105150521
- added J4: Conn_01x02, Connector_PinHeader_2.54mm:PinHeader_1x02_P2.54mm_Vertical, F.Cu at (125.9, 63.0)
- added J5: Conn_02x13_Odd_Even, Connector_PinHeader_2.54mm:PinHeader_2x13_P2.54mm_Vertical, F.Cu at (87.4, 90.7)
- added R36: 5.1k, Resistor_SMD:R_0603_1608Metric, B.Cu at (148.0, 100.0)
- added R37: 1, Resistor_SMD:R_1206_3216Metric, F.Cu at (99.2, 91.8)
- added R38: 1, Resistor_SMD:R_1206_3216Metric, F.Cu at (108.0, 91.9)
- added R39: 1, Resistor_SMD:R_1206_3216Metric, F.Cu at (118.5, 91.9)
- added U8: 629722000214, v3s:629722000214, F.Cu at (149.3, 98.8)
- C21, C22, C23, C34, C41, C54, C56, C8: moved to B.Cu
- C35: value 100n -> 1u
- R8: value 200k 1% -> 5.1k; moved to B.Cu
- moved J1 199.2 mm to (86.4, 102.9), turned to 90 degrees
- moved R6 153.2 mm to (100.6, 57.6), turned to 180 degrees
- moved R7 149.6 mm to (104.5, 61.8), turned to 90 degrees
- moved C8 138.7 mm to (112.3, 61.7), turned to 90 degrees
- moved C29 136.4 mm to (92.0, 94.9), turned to -90 degrees
- moved C21 128.1 mm to (97.4, 104.5), turned to 180 degrees
- moved R9 124.8 mm to (95.1, 103.8), turned to -90 degrees
- moved R10 124.2 mm to (105.7, 103.8), turned to -90 degrees
- moved C22 122.2 mm to (108.0, 104.6), turned to 180 degrees
- moved C14 122.2 mm to (100.0, 102.2), turned to 90 degrees
- moved R13 121.6 mm to (108.0, 104.6), turned to 180 degrees
- moved R8 120.8 mm to (148.0, 97.0)
- moved R14 120.8 mm to (118.5, 104.5), turned to 180 degrees
- moved C27 119.9 mm to (110.5, 94.9), turned to -90 degrees
- moved R27 118.9 mm to (134.0, 103.0), turned to -90 degrees
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Connections:
- net Net-(C18-Pad2) renamed /Power/SW_33
- net Net-(C19-Pad2) renamed /Power/SW_18
- net Net-(C20-Pad2) renamed /Power/SW_12
- C21 pad 1: +3V3 -> Net-(C21-Pad1)
- C22 pad 1: +1V8 -> Net-(C22-Pad1)
- C23 pad 1: +1V2 -> Net-(C23-Pad1)
- C26 pad 1: +3V3 -> Net-(C21-Pad1)
- C27 pad 1: +1V8 -> Net-(C22-Pad1)
- C28 pad 1: +1V2 -> Net-(C23-Pad1)
- C29 pad 1: +3V3 -> Net-(C21-Pad1)
- C30 pad 1: +1V8 -> Net-(C22-Pad1)
- C31 pad 1: +1V2 -> Net-(C23-Pad1)
- J3 pad 1: unconnected-(J3-Pad1) -> CPU_PE0
- J3 pad 10: unconnected-(J3-Pad10) -> CPU_PE9
- J3 pad 11: unconnected-(J3-Pad11) -> CPU_PE10
- J3 pad 12: unconnected-(J3-Pad12) -> CPU_PE11
- J3 pad 13: unconnected-(J3-Pad13) -> CPU_PE12
- J3 pad 14: unconnected-(J3-Pad14) -> CPU_PE13
- J3 pad 15: unconnected-(J3-Pad15) -> CPU_PE14
- J3 pad 16: unconnected-(J3-Pad16) -> CPU_PE15
- J3 pad 17: unconnected-(J3-Pad17) -> CPU_PE16
- J3 pad 18: unconnected-(J3-Pad18) -> CPU_PE17
- J3 pad 19: unconnected-(J3-Pad19) -> CPU_PE18
- J3 pad 2: unconnected-(J3-Pad2) -> CPU_PE1
- J3 pad 20: unconnected-(J3-Pad20) -> CPU_PE19
- J3 pad 21: unconnected-(J3-Pad21) -> CPU_PE20
- J3 pad 22: unconnected-(J3-Pad22) -> CPU_PE21
- J3 pad 23: unconnected-(J3-Pad23) -> CPU_PE22
- J3 pad 24: unconnected-(J3-Pad24) -> CPU_PE23
- J3 pad 25: unconnected-(J3-Pad25) -> CPU_PE24
- J3 pad 26: unconnected-(J3-Pad26) -> GND
- J3 pad 3: unconnected-(J3-Pad3) -> CPU_PE2
- J3 pad 4: unconnected-(J3-Pad4) -> CPU_PE3
- J3 pad 5: unconnected-(J3-Pad5) -> CPU_PE4
- J3 pad 6: unconnected-(J3-Pad6) -> CPU_PE5
- J3 pad 7: unconnected-(J3-Pad7) -> CPU_PE6
- J3 pad 8: unconnected-(J3-Pad8) -> CPU_PE7
- J3 pad 9: unconnected-(J3-Pad9) -> CPU_PE8
- L1 pad 2: +3V3 -> Net-(C21-Pad1)
- L2 pad 2: +1V8 -> Net-(C22-Pad1)
- L3 pad 2: +1V2 -> Net-(C23-Pad1)
- R12 pad 1: +3V3 -> Net-(C21-Pad1)
- R13 pad 1: +1V8 -> Net-(C22-Pad1)
- R14 pad 1: +1V2 -> Net-(C23-Pad1)
- R8 pad 1: +3V3 -> Net-(R8-Pad1)
- R8 pad 2: /CPU/LRADC -> GND
- U1 pad 1: /CPU/CPU_PG4 -> CPU_PG4
- U1 pad 10: /CPU/CPU_PE20 -> CPU_PE20
- U1 pad 11: /CPU/CPU_PE19 -> CPU_PE19
- U1 pad 112: /CPU/LRADC -> unconnected-(U1-Pad112)
- U1 pad 128: /CPU/CPU_PG5 -> CPU_PG5
- U1 pad 13: /CPU/CPU_PE18 -> CPU_PE18
- U1 pad 14: /CPU/CPU_PE17 -> CPU_PE17
- U1 pad 15: /CPU/CPU_PE16 -> CPU_PE16
- U1 pad 16: /CPU/CPU_PE15 -> CPU_PE15
- U1 pad 17: /CPU/CPU_PE14 -> CPU_PE14
- U1 pad 18: /CPU/CPU_PE13 -> CPU_PE13
- U1 pad 2: /CPU/CPU_PG3 -> CPU_PG3
- U1 pad 22: /CPU/CPU_PE12 -> CPU_PE12
- U1 pad 23: /CPU/CPU_PE11 -> CPU_PE11
- U1 pad 24: /CPU/CPU_PE10 -> CPU_PE10
- U1 pad 27: /CPU/CPU_PE9 -> CPU_PE9
- U1 pad 28: /CPU/CPU_PE8 -> CPU_PE8
- U1 pad 3: /CPU/CPU_PG2 -> CPU_PG2
- U1 pad 30: /CPU/CPU_PE7 -> CPU_PE7
- U1 pad 31: /CPU/CPU_PE6 -> CPU_PE6
- U1 pad 32: /CPU/CPU_PE5 -> CPU_PE5
- U1 pad 33: /CPU/CPU_PE4 -> CPU_PE4
- U1 pad 34: /CPU/CPU_PE3 -> CPU_PE3
- U1 pad 35: /CPU/CPU_PE2 -> CPU_PE2
- U1 pad 36: /CPU/CPU_PE1 -> CPU_PE1
- U1 pad 37: /CPU/CPU_PE0 -> CPU_PE0
- U1 pad 39: /CPU/CPU_PB0 -> CPU_PB0
- U1 pad 4: /CPU/CPU_PG1 -> CPU_PG1
- U1 pad 40: /CPU/CPU_PB1 -> CPU_PB1
- U1 pad 41: /CPU/CPU_PB2 -> CPU_PB2
- U1 pad 42: /CPU/CPU_PB3 -> CPU_PB3
- U1 pad 43: /CPU/CPU_PB4 -> CPU_PB4
- U1 pad 44: /CPU/CPU_PB5 -> CPU_PB5
- U1 pad 45: /CPU/CPU_PB6 -> CPU_PB6
- U1 pad 46: /CPU/CPU_PB7 -> CPU_PB7
- U1 pad 5: /CPU/CPU_PG0 -> CPU_PG0
- U1 pad 52: /CPU/CPU_PC0 -> CPU_PC0
- U1 pad 53: /CPU/CPU_PC1 -> CPU_PC1
- U1 pad 54: /CPU/CPU_PC2 -> CPU_PC2
- U1 pad 55: /CPU/CPU_PC3 -> CPU_PC3
- U1 pad 6: /CPU/CPU_PE24 -> CPU_PE24
- U1 pad 7: /CPU/CPU_PE23 -> CPU_PE23
- U1 pad 8: /CPU/CPU_PE22 -> CPU_PE22
- U1 pad 9: /CPU/CPU_PE21 -> CPU_PE21
Routing:
- net +3V3: track 1.19 -> 165.7 mm, vias 1 -> 14
- net +1V2: track 3.38 -> 111.7 mm, vias 0 -> 13
- net /CPU/ETH_SPD: track 0.00 -> 45.8 mm, vias 0 -> 1
- net /CPU/MMC0_CMD: track 0.00 -> 42.7 mm, vias 0 -> 1
- net /CPU/MMC0_D1: track 0.00 -> 42.4 mm, vias 0 -> 1
- net /CPU/MMC0_D2: track 0.00 -> 42.3 mm, vias 0 -> 1
- net /CPU/MMC0_D3: track 0.00 -> 42.2 mm, vias 0 -> 1
- net /CPU/MMC0_D0: track 0.00 -> 41.5 mm, vias 0 -> 1
- net /CPU/ETH_LINK: track 0.00 -> 40.8 mm, vias 0 -> 1
- net /CPU/MMC0_CLK: track 0.00 -> 39.0 mm
- net /CPU/ETH_TXP: track 6.87 -> 44.9 mm, vias 0 -> 1
- net /CPU/ETH_TXN: track 7.28 -> 42.1 mm, vias 0 -> 1
- net CPU_PC2: track 0.00 -> 30.6 mm, vias 0 -> 1
- net CPU_PB4: track 0.00 -> 30.3 mm, vias 0 -> 1
- net CPU_PB6: track 0.00 -> 30.1 mm, vias 0 -> 1
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- added copper zone on F.Cu, net +12V
- added copper zone on In1.Cu, net +12V
- added copper zone on F.Cu, net +1V8
- added copper zone on F.Cu, net /Power/SW_12
- added copper zone on F.Cu, net /Power/SW_18
- added copper zone on F.Cu, net /Power/SW_33
- added copper zone on B.Cu, net GND
- added copper zone on F.Cu, net GND
- added copper zone on F.Cu, net Net-(C21-Pad1)
- added copper zone on F.Cu, net Net-(C22-Pad1)
- added copper zone on F.Cu, net Net-(C23-Pad1)
- added copper zone on F.Cu, net Net-(C4-Pad2)
Other:
- board size 70 x 49 mm -> 70 x 50 mm

Commit message: updates, finish layout, remove usb-uart
Parts:
- removed C60, C68: 4.7u, Capacitor_SMD:C_0603_1608Metric
- removed C61, C69: 100n, Capacitor_SMD:C_0603_1608Metric
- removed D2: RED, LED_SMD:LED_0805_2012Metric
- removed R20: 22.1K, Resistor_SMD:R_0603_1608Metric
- removed R21: 47.5k, Resistor_SMD:R_0603_1608Metric
- removed R22, R23, R26, R27: 1k, Resistor_SMD:R_0603_1608Metric
- removed R24, R25: 0, Resistor_SMD:R_0603_1608Metric
- removed R36, R8: 5.1k, Resistor_SMD:R_0603_1608Metric
- removed U7: CP2102N-Axx-xQFN20, Package_DFN_QFN:SiliconLabs_QFN-20-1EP_3x3mm_P0.5mm_EP1.8x1.8mm
- removed U8: 629722000214, v3s:629722000214
- added J2: Conn_01x06, Connector_JST:JST_PH_B6B-PH-K_1x06_P2.00mm_Vertical, F.Cu at (146.0, 96.3)
- D1: value RED -> D_Small; footprint LED_SMD:LED_0805_2012Metric -> Diode_SMD:D_SMA
- L1, L2, L3: value NRS6045T6R8MMGK -> VLS6045AF-6R8M
- Y1: value SC32S-7PF20PPM -> Q13FC1350000212; footprint v3s:SC32S-7PF20PPM -> Crystal:Crystal_SMD_3215-2Pin_3.2x1.5mm
- moved D1 49.0 mm to (89.1, 102.9), turned to 180 degrees
- moved R6 15.7 mm to (115.6, 62.1), turned to -90 degrees
- moved J1 4.62 mm to (87.1, 98.3)
- moved D3 3.32 mm to (126.8, 102.9), turned to 0 degrees
- moved C34 2.94 mm to (100.4, 82.8), turned to 180 degrees
- moved C32 1.52 mm to (102.4, 72.5)
- moved J4 1.30 mm to (125.9, 61.8)
- moved C57 0.60 mm to (112.1, 67.5)
- moved C3 0.42 mm to (114.0, 62.1)
- moved C55 0.42 mm to (111.5, 71.4)
- moved Y1 0.08 mm to (119.6, 64.0), turned to -90 degrees
Connections:
- D1 pad 1: Net-(D1-Pad1) -> +12V
- D1 pad 2: +3V3 -> Net-(J1-Pad1)
- D3 pad 2: /DebugUART/USB_VCC -> Net-(D3-Pad2)
- J1 pad 1: +12V -> Net-(J1-Pad1)
Routing:
- net +3V3: track 165.7 -> 231.6 mm, vias 14 -> 15
- net GND: track 1.21 -> 48.7 mm, vias 1 -> 37
- net /CPU/UART0_RX: track 1.76 -> 42.8 mm
- net +3V0: track 6.68 -> 45.9 mm, vias 1 -> 4
- net /CPU/UART0_TX: track 3.02 -> 41.7 mm
- net Net-(D3-Pad2): track 0.00 -> 20.9 mm
- net +1V8: track 27.7 -> 44.5 mm, vias 6 -> 8
- net /CPU/CPU_RESET: track 2.59 -> 18.7 mm, vias 1 -> 2
- net /DebugUART/USB_D+: track 14.1 -> 0.00 mm, vias 2 -> 0
- net /DebugUART/USB_D-: track 12.4 -> 0.00 mm
- net /DebugUART/USB_VBUS_DETECT: track 7.31 -> 0.00 mm, vias 2 -> 0
- net Net-(C60-Pad1): track 7.16 -> 0.00 mm
- net Net-(J1-Pad1): track 0.00 -> 4.58 mm
- net Net-(R22-Pad1): track 4.55 -> 0.00 mm
- net Net-(R24-Pad1): track 4.40 -> 0.00 mm
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- added copper zone on In1.Cu, net GND
- added copper zone on In2.Cu, net GND
Other:
- board text added: "+3V3"
- board text added: "+VIN"
- board text added: "+Vcc"
- board text added: "1"
- board text added: "2"
- board text added: "3"
- board text added: "4"
- board text added: "GND"
- board text added: "RESET"
- board text added: "UART0_RX"
- board text added: "UART0_TX"
